File: hw/ESP32_PRELIM_DESIGN.kicad_sch (KiCad schematic)
At the start: 12 parts, among them J1 Conn_01x09_Pin, J2 USB_C_Receptacle_USB2.0_16P, M1 Motor_DC, U1 ESP32-S3-WROOM-1, U2 DRV2605LDGS, U3 TPD2EUSB30A

Commit message: updated schema
Parts:
- removed J2: USB_C_Receptacle_USB2.0_16P, symbol Connector:USB_C_Receptacle_USB2.0_16P
- removed U3: TPD2EUSB30A, Package_TO_SOT_SMD:Texas_DRT-3, symbol Power_Protection:TPD2EUSB30A
Changed lines of the file:
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@@
-	)
-	(symbol
-		(lib_id "Connector:USB_C_Receptacle_USB2.0_16P")
-		(at 241.3 62.23 180)
-		(unit 1)
-		(body_style 1)
-		(exclude_from_sim no)
-		(in_bom yes)
-		(on_board yes)
-		(in_pos_files yes)
-		(dnp no)
-		(fields_autoplaced yes)
-		(property "Reference" "J2"
-			(at 252.73 60.9599 0)
-			(show_name no)
-			(do_not_autoplace no)
-			(effects
-				(font
-					(size 1.27 1.27)
-				)
-				(justify right)
-			)
-		)
-		(property "Value" "USB_C_Receptacle_USB2.0_16P"
-			(at 252.73 63.4999 0)
-			(show_name no)
-			(do_not_autoplace no)
-			(effects
-				(font
-					(size 1.27 1.27)
-				)
-				(justify right)
-			)
-		)
-		(property "Footprint" ""
-			(at 237.49 62.23 0)
-			(hide yes)
-			(show_name no)
-			(do_not_autoplace no)
-			(effects
-				(font
-					(size 1.27 1.27)
-				)
-			)
-		)
-		(property "Datasheet" "https://www.usb.org/sites/default/files/documents/usb_type-c.zip"
-			(at 237.49 62.23 0)
-			(hide yes)
-			(show_name no)
-			(do_not_autoplace no)
-			(effects
-				(font
-					(size 1.27 1.27)
-				)
-			)
-		)
-		(property "Description" "USB 2.0-only 16P Type-C Receptacle connector"
-			(at 241.3 62.23 0)
-			(hide yes)
-			(show_name no)
-			(do_not_autoplace no)
-			(effects
-				(font
-					(size 1.27 1.27)
-				)
-			)
-		)
-		(pin "B5"
-		)
-		(pin "SH"
-		)
-		(pin "B7"
-		)
-		(pin "B12"
-		)
-		(pin "B9"
-		)
-		(pin "B8"
-		)
-		(pin "B6"
-		)
-		(pin "B4"
-		)
-		(pin "A1"
-		)
-		(pin "A9"
-		)
-		(pin "A4"
-		)
-		(pin "A5"
-		)
-		(pin "A6"
-		)
-		(pin "A7"
-		)
-		(pin "A8"
-		)
-		(pin "A12"
-		)
-		(pin "B1"
-		)
-		(instances
-			(project "ESP32_PRELIM_DESIGN"
-				(path "/ad7b4e31-bbaa-4804-aa31-814eb5fa2fbb"
-					(reference "J2")
-					(unit 1)
-				)
-			)
-		)
 	)
 	(symbol
@@
 					(unit 1)
 				)
-			)
-		)
-	)
-	(symbol
-		(lib_id "Power_Protection:TPD2EUSB30A")
-		(at 207.01 66.04 0)
-		(unit 1)
-		(body_style 1)
-		(exclude_from_sim no)
-		(in_bom yes)
-		(on_board yes)
-		(in_pos_files yes)
-		(dnp no)
-		(fields_autoplaced yes)
-		(property "Reference" "U3"
-			(at 207.01 55.88 0)
-			(show_name no)
-			(do_not_autoplace no)
-			(effects
-				(font
-					(size 1.27 1.27)
-				)
-			)
-		)
-		(property "Value" "TPD2EUSB30A"
-			(at 207.01 58.42 0)
-			(show_name no)
-			(do_not_autoplace no)
-			(effects
-				(font
-					(size 1.27 1.27)
-				)
-			)
-		)
-		(property "Footprint" "Package_TO_SOT_SMD:Texas_DRT-3"
-			(at 187.96 73.66 0)
-			(hide yes)
-			(show_name no)
-			(do_not_autoplace no)
-			(effects
-				(font
-					(size 1.27 1.27)
-				)
-			)
-		)
-		(property "Datasheet" "http://www.ti.com/lit/ds/symlink/tpd2eusb30a.pdf"
-			(at 207.01 66.04 0)
-			(hide yes)
-			(show_name no)
-			(do_not_autoplace no)
-			(effects
-				(font
-					(size 1.27 1.27)
-				)
-			)
-		)
-		(property "Description" "2-Channel ESD Protection for Super-Speed USB 3.0 Interface, DRT-3"
-			(at 207.01 66.04 0)
-			(hide yes)
-			(show_name no)
-			(do_not_autoplace no)
-			(effects
-				(font
-					(size 1.27 1.27)
-				)
-			)
-		)
-		(pin "2"
-		)
-		(pin "1"
-		)
-		(pin "3"
-		)
-		(instances
-			(project "ESP32_PRELIM_DESIGN"
-				(path "/ad7b4e31-bbaa-4804-aa31-814eb5fa2fbb"
-					(reference "U3")
-					(unit 1)
-				)

Commit message: added setup files for display and haptics integration
Parts:
- added BT2: Battery_Cell, symbol Device:Battery_Cell
- added C10: 2*10uF, symbol Device:C
- added C11: 100nF, symbol Device:C
- added C12: 3*22uF, symbol Device:C
- added C13: 0.1uF, symbol Device:C
- added C14: 10uF, symbol Device:C
- added C15: 1uF, symbol Device:C
- added C16, C17: 4.7uF, symbol Device:C
- added C18: 10k, symbol Device:C
- added J4: Conn_01x02_Pin, symbol Connector:Conn_01x02_Pin
- added J5: USB_C_Receptacle_USB2.0_16P, symbol Connector:USB_C_Receptacle_USB2.0_16P
- added L2: 1.5uH, symbol Device:L
- added R12, R14: 1M, symbol Device:R_US
- added R13: 180k, symbol Device:R_US
- added R15, R16: 5.1k, symbol Device:R_US
- added R17: 1.18k, symbol Device:R_US
- added R18: 1.13k, symbol Device:R_US
- added R19: 10k, symbol Device:R_US
- added U10: BQ24075RGT, Package_DFN_QFN:VQFN-16-1EP_3x3mm_P0.5mm_EP1.6x1.6mm, symbol Battery_Management:BQ24075RGT
- added U7: TPS63020DSJR, TPS63020DSJR:IC_TPS63020DSJR, symbol TPS63020DSJR:TPS63020DSJR
- added U8: MAX17048G_T10, MAX17048G_T10:SON50P200X200X80-9N, symbol MAX17048G_T10:MAX17048G_T10
- added U9: TPD2EUSB30A, Package_TO_SOT_SMD:Texas_DRT-3, symbol Power_Protection:TPD2EUSB30A
Connections:
- net +3.3V: now also C12.1, R12.1, R14.1, U7.4 (VOUT_4), U7.5 (VOUT_5)
- net GND: now also C10.1, C11.1, C12.2, C13.1, C14.2, C15.2, C16.1, C17.1, C18.1, J4.2 (Pin_2), J5.A1 (GND), J5.A12 (GND), J5.B1 (GND), J5.B12 (GND), J5.SH (SHIELD), R13.2, R15.2, R16.2, R17.2, R18.2, R19.2, U10.14 (TMR), U10.17 (VSS), U10.4 (~{CE}), U10.6 (EN1), U10.8 (VSS), U7.15 (PGND), U7.2 (GND), U8.1 (CTG), U8.4 (GND), U8.6 (QSTRT), U8.9 (EP), U9.3 (GND)
- net SCL: now also U8.7 (SCL)
- net SDA: now also U8.8 (SDA)
- new net: C11.2, U7.1 (VINA), U7.12 (EN), U7.13 (PS/SYNC)
- new net: J5.A5 (CC1), R16.1
- new net: J5.B5 (CC2), R15.1
- new net: R19.1, U10.1 (TS)
- new net: R17.1, U10.12 (ILIM)
- new net: R18.1, U10.16 (ISET)
- new net: R12.2, R13.1, U7.3 (FB)
- new net: C18.2, U8.5 (~{ALERT})
- new net: L2.1, U7.8 (L1_8), U7.9 (L1_9)
- new net: L2.2, U7.6 (L2_6), U7.7 (L2_7)
- new net: R14.2, U7.14 (PG)
- new net +5V: C14.1, C15.1, J5.A4 (VBUS), J5.A9 (VBUS), J5.B4 (VBUS), J5.B9 (VBUS), U10.13 (IN)
- new net USB_DM: J5.A7 (D-), J5.B7 (D-), U9.2 (D-)
- new net USB_DP: J5.A6 (D+), J5.B6 (D+), U9.1 (D+)
- new net VBAT: C13.2, C17.2, J4.1 (Pin_1), U10.2 (BAT), U10.3 (BAT), U8.2 (CELL), U8.3 (VDD)
- new net VSYS: C10.2, C16.2, U10.10 (OUT), U10.11 (OUT), U10.5 (EN2), U7.10 (VIN_10), U7.11 (VIN_11)
- no-connect marks 1 -> 5
Other:
- note added: "JST_PH 2 connector for battery"
- note added: "add buttons for boot and reset"
- note added: "decide gpio for ALRT"
- note added: "for reference jst_PH connect connects to the battery need to add all footprints after"
- note removed: "JST PH COnnector to use to battery"
