File: hardware/ESP32_PRELIM_DESIGN.kicad_pcb (KiCad board)
At the start: 4 copper layers, 66 x 40 mm, 79 parts, among them J1 Conn_01x11_Socket, J4 Conn_01x02_Pin, J5 USB_C_Receptacle_USB2.0_16P, J6 Conn_01x05_Pin, J7 Conn_01x05_Pin, Q1 2N7002, SW1 SW_Push, SW2 SW_Push, SW3 SW_Push, U1 ESP32-S3-WROOM-1, U10 BQ24075RGT, U11 MAX98357A, U12 USBLC6-2SC6, U2 DRV2605LDGS, U3 TPS63020DSJR, U4 MAX17048G_T10

Commit message: final changes befpre pcb rev submission
Parts:
- R18: value 1.78k -> 2k
Routing:
- net +3.3V: track 184.3 -> 185.5 mm
- net /USB_DP: track 37.7 -> 38.5 mm
- net GND: vias 47 -> 49
Changed lines of the file:
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@@
 		(capping no)
 		(filling no)
-		(zone_defaults)
 		(pcbplotparams
 			(layerselection 0x00000000_00000000_55555555_5755f5ff)
@@
 			)
 		)
-		(property "Value" "1.78k"
+		(property "Value" "2k"
 			(at 0 1.65 0)
 			(layer "F.Fab")
@@
 	)
 	(via
+		(at 222.8 120.6)
+		(size 0.6)
+		(drill 0.3)
+		(layers "F.Cu" "B.Cu")
+		(free yes)
+		(net "GND")
+	)
+	(via
 		(at 223.3 132.7)
 		(size 0.6)
@@
 	)
 	(via
+		(at 209.5 115.6)
+		(size 0.6)
+		(drill 0.3)
+		(layers "F.Cu" "B.Cu")
+		(free yes)
+		(net "GND")
+	)
+	(via
 		(at 228.38 122.48)
 		(size 0.6)
@@
 	)
 	(segment
-		(start 208.375 101.7)
-		(end 206.6375 101.7)
-		(width 0.3)
-		(layer "F.Cu")
-		(net "+3.3V")
-	)
-	(segment
 		(start 198.8 121.6)
 		(end 198.8 117.465)
@@
 	)
 	(segment
-		(start 208.4 101.725)
-		(end 208.375 101.7)
-		(width 0.2)
-		(layer "F.Cu")
-		(net "+3.3V")
-	)
-	(segment
 		(start 232.74 118.73)
 		(end 233.9625 119.9525)
@@
 	)
 	(segment
+		(start 208 101.7)
+		(end 206.6375 101.7)
+		(width 0.3)
+		(layer "F.Cu")
+		(net "+3.3V")
+	)
+	(segment
 		(start 211.25 102.76)
 		(end 208.4025 102.76)
@@
 	)
 	(via
-		(at 208.4 101.725)
+		(at 208 101.7)
 		(size 0.6)
 		(drill 0.3)
@@
 	)
 	(segment
+		(start 207.975 101.725)
+		(end 204.975 101.725)
+		(width 0.3)
+		(layer "In2.Cu")
+		(net "+3.3V")
+	)
+	(segment
 		(start 194.5 126.95)
 		(end 196.6 126.95)
@@
 	)
 	(segment
+		(start 203.075 103.625)
+		(end 203.075 112.25)
+		(width 0.3)
+		(layer "In2.Cu")
+		(net "+3.3V")
+	)
+	(segment
 		(start 228.29 121.2)
 		(end 231.81 117.68)
@@
 	)
 	(segment
-		(start 203.075 107.05)
-		(end 203.075 112.25)
-		(width 0.3)
-		(layer "In2.Cu")
-		(net "+3.3V")
-	)
-	(segment
 		(start 210.3625 135.2375)
 		(end 212.9 132.7)
@@
 	)
 	(segment
-		(start 208.4 101.725)
-		(end 203.075 107.05)
+		(start 208 101.7)
+		(end 207.975 101.725)
 		(width 0.3)
 		(layer "In2.Cu")
@@
 	)
 	(segment
+		(start 204.975 101.725)
+		(end 203.075 103.625)
+		(width 0.3)
+		(layer "In2.Cu")
+		(net "+3.3V")
+	)
+	(segment
 		(start 225.85 132.725)
 		(end 227.075 133.95)
@@
 	)
 	(segment
+		(start 209.4 117.525003)
+		(end 210.092979 117.525003)
+		(width 0.2)
+		(layer "F.Cu")
+		(net "/USB_DP")
+	)
+	(segment
 		(start 189.7125 109.5)
 		(end 191.4875 109.5)
@@
 	)
 	(segment
-		(start 211.25 118)
-		(end 209.68 118)
+		(start 210.092979 117.525003)
+		(end 210.567976 118)
 		(width 0.2)
 		(layer "F.Cu")
@@
 		(net "/USB_DP")
 	)
+	(segment
+		(start 210.567976 118)
+		(end 211.25 118)
+		(width 0.2)
+		(layer "F.Cu")
+		(net "/USB_DP")
+	)
 	(via
 		(at 186.3 111.8)
@@
 	)
 	(via
-		(at 209.68 118)
+		(at 209.4 117.525003)
 		(size 0.6)
 		(drill 0.3)
@@
 	)
 	(segment
-		(start 188.8625 111.778185)
-		(end 188.8625 110.35)
+		(start 209.4 117.525003)
+		(end 209.4 118.28)
 		(width 0.2)
 		(layer "B.Cu")
@@
 	)
 	(segment
-		(start 186.3 111.8)
-		(end 188.35 109.75)
+		(start 188.8625 110.35)
+		(end 189.4625 109.75)
 		(width 0.2)
 		(layer "B.Cu")
@@
 	)
 	(segment
-		(start 188.8625 110.35)
-		(end 189.4625 109.75)
+		(start 209.4 118.28)
+		(end 208.84 118.84)
+		(width 0.2)
+		(layer "B.Cu")
+		(net "/USB_DP")
+	)
+	(segment
+		(start 186.3 111.8)
+		(end 188.35 109.75)
 		(width 0.2)
 		(layer "B.Cu")
@@
 	)
 	(segment
-		(start 209.68 118)
-		(end 208.84 118.84)
+		(start 188.8625 111.778185)
+		(end 188.8625 110.35)
 		(width 0.2)
 		(layer "B.Cu")
@@
 	)
 	(segment
-		(start 193.75 113.715)
-		(end 193.75 112.553076)
-		(width 0.2)
-		(layer "F.Cu")
-		(net "/SDA")
-	)
-	(segment
-		(start 209.132941 115.46)
-		(end 206.6 112.927059)
+		(start 211.25 115.46)
+		(end 210.79 115)
 		(width 0.2)
 		(layer "F.Cu")
@@
 	)
 	(segment
-		(start 206.6 112.927059)
-		(end 206.6 112.25)
+		(start 193.75 113.715)
+		(end 193.75 112.553076)
 		(width 0.2)
 		(layer "F.Cu")
@@
 	)
 	(segment
-		(start 197.45 103.5)
-		(end 198.641724 103.5)
+		(start 210.79 115)
+		(end 208.672941 115)
 		(width 0.2)
 		(layer "F.Cu")
@@
 	)
 	(segment
-		(start 211.25 115.46)
-		(end 209.132941 115.46)
+		(start 206.6 112.927059)
+		(end 206.6 112.25)
+		(width 0.2)
+		(layer "F.Cu")
+		(net "/SDA")
+	)
+	(segment
+		(start 197.45 103.5)
+		(end 198.641724 103.5)
 		(width 0.2)
 		(layer "F.Cu")
@@
 		(net "/SDA")
 	)
+	(segment
+		(start 208.672941 115)
+		(end 206.6 112.927059)
+		(width 0.2)
+		(layer "F.Cu")
+		(net "/SDA")
+	)
 	(via
 		(at 193.454244 112.25732)
@@
 	(segment
 		(start 208.46147 113.94)
-		(end 208.71147 114.19)
+		(end 209.12147 114.6)
 		(width 0.2)
 		(layer "F.Cu")
@@
 	)
 	(segment
+		(start 209.12147 114.6)
+		(end 210.84 114.6)
+		(width 0.2)
+		(layer "F.Cu")
+		(net "/FG_ALRT")
+	)
+	(segment
 		(start 195.76 113.715)
 		(end 196.45 113.715)
@@
 	)
 	(segment
-		(start 208.71147 114.19)
+		(start 210.84 114.6)
 		(end 211.25 114.19)
 		(width 0.2)
@@
 	)
 	(segment
-		(start 223.044785 121.595215)
-		(end 227.999571 126.55)
+		(start 220.635 120.58)
+		(end 221.255 121.2)
 		(width 0.2)
 		(layer "F.Cu")
@@
 	)
 	(segment
-		(start 220.635 120.58)
-		(end 220.635 119.25)
+		(start 220.635 119.25)
+		(end 220.635 120.58)
 		(width 0.2)
 		(layer "F.Cu")
@@
 	)
 	(segment
-		(start 221.650215 121.595215)
-		(end 223.044785 121.595215)
+		(start 222.649571 121.2)
+		(end 227.999571 126.55)
 		(width 0.2)
 		(layer "F.Cu")
@@
 	)
 	(segment
-		(start 220.635 120.58)
-		(end 221.650215 121.595215)
+		(start 227.999571 126.55)
+		(end 242.28 126.55)
 		(width 0.2)
 		(layer "F.Cu")
@@
 	)
 	(segment
-		(start 227.999571 126.55)
-		(end 242.28 126.55)
+		(start 221.255 121.2)
+		(end 222.649571 121.2)
 		(width 0.2)
 		(layer "F.Cu")
@@
 	)
 	(segment
-		(start 223.175 121.159744)
+		(start 223.7 120.3)
+		(end 223.7 121.684744)
+		(width 0.2)
+		(layer "F.Cu")
+		(net "/OLED_RST")
+	)
+	(segment
+		(start 223.7 121.684744)
 		(end 228.165256 126.15)
 		(width 0.2)
@@
 	)
 	(segment
+		(start 223.695 119.77)
+		(end 223.695 120.295)
+		(width 0.2)
+		(layer "F.Cu")
+		(net "/OLED_RST")
+	)
+	(segment
+		(start 223.695 120.295)
+		(end 223.7 120.3)
+		(width 0.2)
+		(layer "F.Cu")
+		(net "/OLED_RST")
+	)
+	(segment
 		(start 223.175 119.25)
-		(end 223.175 121.159744)
+		(end 223.695 119.77)
 		(width 0.2)
 		(layer "F.Cu")
