File: hardware/ESP32_PRELIM_DESIGN.kicad_pcb (KiCad board)
At the start: 4 copper layers, 66 x 40 mm, 79 parts, among them J1 Conn_01x11_Socket, J4 Conn_01x02_Pin, J5 USB_C_Receptacle_USB2.0_16P, J6 Conn_01x05_Pin, J7 Conn_01x05_Pin, Q1 2N7002, SW1 SW_Push, SW2 SW_Push, SW3 SW_Push, U1 ESP32-S3-WROOM-1, U10 BQ24075RGT, U11 MAX98357A, U12 USBLC6-2SC6, U2 DRV2605LDGS, U3 TPS63020DSJR, U4 MAX17048G_T10

Commit message: final changes before CDR
Parts:
- renumbered C18 to C1, C13 to C10, C24 to C11, C10 to C12, C11 to C13, C22 to C16, C12 to C17, C16 to C18, C23 to C19, C27 to C2, C17 to C20, C28 to C3, C20 to C4, C1 to C5, C21 to C6, C26 to C7, C19 to C8, C25 to C9, D5 to D1, D4 to D2, D1 to D3, D2 to D4, D3 to D5, TP8 to FG_ALRT1, TP5 to GND1, J4 to J1, J1 to J2, J7 to J3, J6 to J4, L2 to L1, R2 to R1, R22 to R10, R6 to R11, R29 to R12, R28 to R13, R27 to R14, R12 to R19, R1 to R2, R19 to R20, R13 to R21, R25 to R22, R14 to R23, R4 to R24, R26 to R25, R5 to R26, R23 to R3, R30 to R4, R7 to R5, R24 to R6, R3 to R7, R20 to R8, R21 to R9, TP2 to RX1, TP7 to SCL1, TP6 to SDA1, TP3 to TP1, TP4 to TP2, TP1 to TX1, U2 to U1, U1 to U2, U11 to U3, U12 to U5, U3 to U6, U10 to U7
Routing:
- net /VSYS: track 138.2 -> 140.7 mm
