File: hardware/ESP32_PRELIM_DESIGN.kicad_pcb (KiCad board)
At the start: 4 copper layers, 66 x 40 mm, 79 parts, among them J1 Conn_01x02_Pin, J2 Conn_01x11_Socket, J3 Conn_01x05_Pin, J4 Conn_01x05_Pin, J5 USB_C_Receptacle_USB2.0_16P, Q1 2N7002, SW1 SW_Push, SW2 SW_Push, SW3 SW_Push, U1 DRV2605LDGS, U2 ESP32-S3-WROOM-1, U3 MAX98357A, U4 MAX17048G_T10, U5 USBLC6-2SC6, U6 TPS63020DSJR, U7 BQ24075RGT

Commit message: final push (pk verified)
Parts:
- added H3: MountingHole, MountingHole:MountingHole_2.2mm_M2, F.Cu at (237.6, 128.1)
- R17: value 1.18k -> 3.3k
- moved C11 8.77 mm to (193.8, 128.2), turned to -90 degrees
- moved R24 8.17 mm to (239.2, 114.8), turned to 0 degrees
- moved R26 6.10 mm to (239.2, 112.8), turned to 0 degrees
- moved D4 5.56 mm to (235.5, 114.8), turned to 0 degrees
- moved D5 4.49 mm to (235.5, 112.8), turned to 0 degrees
- moved R11 3.36 mm to (239.2, 116.7), turned to 180 degrees
- moved D2 3.16 mm to (235.5, 116.7), turned to 0 degrees
- moved R5 3.15 mm to (239.2, 118.7), turned to 180 degrees
- moved R25 3.00 mm to (198.6, 125.8)
- moved D1 2.66 mm to (235.5, 118.7), turned to 0 degrees
- moved C5 2.40 mm to (205.5, 104.1)
- moved C6 2.40 mm to (205.6, 101.7)
Connections:
- C13 pad 2: Net-(U6-VINA) -> /VSYS
- R24 pad 2: /VSYS -> +3.3V
- R26 pad 2: /VSYS -> +3.3V
- U6 pad 1: Net-(U6-VINA) -> /VSYS
- U6 pad 11: Net-(U6-VINA) -> /VSYS
Routing:
- net +3.3V: track 185.5 -> 164.2 mm, vias 7 -> 8
- net /SCL: track 61.3 -> 45.3 mm, vias 4 -> 3
- net Net-(U6-VINA): track 12.3 -> 0.00 mm, vias 2 -> 0
- net /VSYS: track 140.7 -> 150.9 mm, vias 6 -> 8
- net GND: track 35.9 -> 42.5 mm, vias 49 -> 59
- net /CHG_STAT: track 57.4 -> 62.9 mm
- net /PGOOD: track 57.3 -> 62.3 mm
- net Net-(U6-L1_8): track 5.46 -> 0.50 mm
- net Net-(U2-IO48): track 18.3 -> 22.3 mm
- net /I2S_BCLK: track 29.2 -> 28.0 mm
- net Net-(U6-EN): track 19.9 -> 21.0 mm, vias 0 -> 2
- net /I2S_DOUT: track 31.3 -> 30.6 mm
- net /VBUS: track 22.5 -> 23.2 mm
- added copper zone on F.Cu, net Net-(U6-L1_8)
- added copper zone on F.Cu, net Net-(U6-L2_6)

Commit message: final check before fabrication
Parts:
- added C21: 10uF, Capacitor_SMD:C_0805_2012Metric_Pad1.18x1.45mm_HandSolder, F.Cu at (203.0, 129.7)
- added D6: BAT54WS, Diode_SMD:D_SOD-323_HandSoldering, F.Cu at (203.0, 127.2)
Connections:
- net Net-(U6-EN) renamed /U6_EN
Routing:
- net /VBUS: track 23.2 -> 37.9 mm, vias 3 -> 5
- net /U6_EN: track 21.0 -> 23.6 mm, vias 2 -> 3
- net GND: track 42.5 -> 43.8 mm, vias 59 -> 60

Commit message: changes after GTA review
Parts:
- moved R9 1.78 mm to (232.2, 103.7), turned to 180 degrees
- moved R8 1.14 mm to (232.4, 101.7), turned to 0 degrees
- moved R10 0.59 mm to (232.2, 105.8)
- moved U4 0.46 mm to (194.1, 114.6)
Routing:
- net GND: track 43.8 -> 42.6 mm, vias 60 -> 59
- net Net-(U3-GAIN_SLOT): track 4.06 -> 5.10 mm
- net Net-(U3-~{SD_MODE}): track 1.14 -> 1.91 mm
- net /FG_ALRT: track 31.7 -> 32.2 mm
