File: hardware/ESP32_PRELIM_DESIGN.kicad_sch (KiCad schematic)
At the start: 35 parts, among them J1 Conn_01x09_Pin, J4 Conn_01x02_Pin, J5 USB_C_Receptacle_USB2.0_16P, M1 Motor_DC, U1 ESP32-S3-WROOM-1, U10 BQ24075RGT, U2 DRV2605LDGS, U7 TPS63020DSJR, U8 MAX17048G_T10, U9 TPD2EUSB30A

Commit message: FINAL SCHEMATIC
finalized schematic and footprints so layout and routing can start
Parts:
- removed BT2: Battery_Cell, symbol Device:Battery_Cell
- removed C18: 10k, symbol Device:C
- removed J1: Conn_01x09_Pin, symbol Connector:Conn_01x09_Pin
- removed U7: TPS63020DSJR, TPS63020DSJR:IC_TPS63020DSJR, symbol TPS63020DSJR:TPS63020DSJR
- removed U8: MAX17048G_T10, MAX17048G_T10:SON50P200X200X80-9N, symbol MAX17048G_T10:MAX17048G_T10
- removed U9: TPD2EUSB30A, Package_TO_SOT_SMD:Texas_DRT-3, symbol Power_Protection:TPD2EUSB30A
- added C19, C28: 0.1uF, Capacitor_SMD:C_0805_2012Metric_Pad1.18x1.45mm_HandSolder, symbol Device:C
- added C20: 1uF, Capacitor_SMD:C_0805_2012Metric_Pad1.18x1.45mm_HandSolder, symbol Device:C
- added C21, C22, C23, C26: 22uF, Capacitor_SMD:C_1206_3216Metric_Pad1.33x1.80mm_HandSolder, symbol Device:C
- added C24, C25: 10uF, Capacitor_SMD:C_0805_2012Metric_Pad1.18x1.45mm_HandSolder, symbol Device:C
- added D1: BAT54C, Package_TO_SOT_SMD:SOT-23, symbol Diode:BAT54C
- added H1, H2, H3, H4: MountingHole, MountingHole:MountingHole_2.2mm_M2, symbol Mechanical:MountingHole
- added J1: Conn_01x11_Socket, Connector_PinSocket_2.54mm:PinSocket_1x11_P2.54mm_Vertical, symbol Connector:Conn_01x11_Socket
- added J6, J7: Conn_01x05_Pin, Connector_JST:JST_PH_S5B-PH-K_1x05_P2.00mm_Horizontal, symbol Connector:Conn_01x05_Pin
- added LS1: Speaker, Connector_Molex:Molex_PicoBlade_53261-0271_1x02-1MP_P1.25mm_Horizontal, symbol Device:Speaker
- added Q1: 2N7002, Package_TO_SOT_SMD:SOT-23, symbol Transistor_FET:2N7002
- added R20, R21: 0, Resistor_SMD:R_0805_2012Metric_Pad1.20x1.40mm_HandSolder, symbol Device:R_US
- added R22: 680k, Resistor_SMD:R_0805_2012Metric_Pad1.20x1.40mm_HandSolder, symbol Device:R_US
- added R23, R24, R25, R26, R29: 10k, Resistor_SMD:R_0805_2012Metric_Pad1.20x1.40mm_HandSolder, symbol Device:R_US
- added R27, R28: 100k, Resistor_SMD:R_0805_2012Metric_Pad1.20x1.40mm_HandSolder, symbol Device:R_US
- added R30: 33, Resistor_SMD:R_0805_2012Metric_Pad1.20x1.40mm_HandSolder, symbol Device:R_US
- added SW1, SW2: SW_Push, Button_Switch_SMD:SW_SPST_CK_KMS2xxGP, symbol Switch:SW_Push
- added SW3: SW_Push, Button_Switch_THT:SW_NKK_GW12LJP, symbol Switch:SW_Push
- added TP1: TX, TestPoint:TestPoint_THTPad_D1.5mm_Drill0.7mm, symbol Connector:TestPoint
- added TP2: RX, TestPoint:TestPoint_THTPad_D1.5mm_Drill0.7mm, symbol Connector:TestPoint
- added TP3, TP4: TestPoint, TestPoint:TestPoint_Pad_1.5x1.5mm, symbol Connector:TestPoint
- added TP5: GND, TestPoint:TestPoint_THTPad_D1.5mm_Drill0.7mm, symbol Connector:TestPoint
- added U11: MAX98357A, Package_DFN_QFN:TQFN-16-1EP_3x3mm_P0.5mm_EP1.23x1.23mm, symbol Audio:MAX98357A
- added U12: USBLC6-2SC6, Package_TO_SOT_SMD:SOT-23-6, symbol Power_Protection:USBLC6-2SC6
- added U3: TPS63020DSJR, SLATE:IC_TPS63020DSJR, symbol TPS63020DSJR:TPS63020DSJR
- added U4: MAX17048G_T10, MAX17048G_T10:SON50P200X200X80-9N, symbol MAX17048G_T10:MAX17048G_T10
- C1, C13, C14, C15, C16, C17: footprint (none) -> Capacitor_SMD:C_0805_2012Metric_Pad1.18x1.45mm_HandSolder
- C10: value 2*10uF -> 10uF; footprint (none) -> Capacitor_SMD:C_0805_2012Metric_Pad1.18x1.45mm_HandSolder
- C11: value 100nF -> 0.1uF; footprint (none) -> Capacitor_SMD:C_0805_2012Metric_Pad1.18x1.45mm_HandSolder
- C12: value 3*22uF -> 22uF; footprint (none) -> Capacitor_SMD:C_1206_3216Metric_Pad1.33x1.80mm_HandSolder
- C18, C27: renamed from 1uF; value C -> 1uF; footprint (none) -> Capacitor_SMD:C_0805_2012Metric_Pad1.18x1.45mm_HandSolder
- J4: footprint (none) -> Connector_JST:JST_PH_S2B-PH-K_1x02_P2.00mm_Horizontal
- J5: footprint (none) -> Connector_USB:USB_C_Receptacle_GCT_USB4105-xx-A_16P_TopMnt_Horizontal
- L2: footprint (none) -> Inductor_SMD:L_Coilcraft_XAL4020-XXX
- M1: now not fitted; now left out of the parts list
- R1, R12, R13, R14, R15, R16, R17, R18, R19, R2, R3: footprint (none) -> Resistor_SMD:R_0805_2012Metric_Pad1.20x1.40mm_HandSolder
- U10: footprint Package_DFN_QFN:VQFN-16-1EP_3x3mm_P0.5mm_EP1.6x1.6mm -> Package_DFN_QFN:QFN-16-1EP_3x3mm_P0.5mm_EP1.7x1.7mm
Connections:
- net +3.3V: now also C21.2, C22.1, C23.1, J1.2 (Pin_2), J6.1 (Pin_1), J7.1 (Pin_1), J7.3 (Pin_3), R23.1, R24.1, R25.1, R26.1, R29.2, U3.4 (VOUT_4), U3.5 (VOUT_5); no longer C27.1, U2.10 (VDD)
- net GND: now also U10.15 (SYSOFF), C19.1, C20.1, C21.1, C22.2, C23.2, C24.1, C25.1, C26.2, C28.1, J1.1 (Pin_1), J6.2 (Pin_2), J6.3 (Pin_3), J7.2 (Pin_2), Q1.2 (S), R21.2, R27.1, R28.1, SW1.2, SW2.2, TP5.1, U11.11 (GND), U11.15 (GND), U11.17 (PAD), U11.3 (GND), U12.2 (GND), U3.13 (PS/SYNC), U3.15 (PGND), U3.2 (GND), U4.1 (CTG), U4.4 (GND), U4.6 (QSTRT), U4.9 (EP); no longer U10.14 (TMR)
- net MISO_SD: now also J1.7 (Pin_7)
- net SCL: now also U4.7 (SCL)
- net SDA: now also U4.8 (SDA)
- net SDCS: now also J1.11 (Pin_11)
- net USB_DM: now also U1.13 (USB_D-), U12.3 (I/O2), U12.4 (I/O2)
- net USB_DP: now also U1.14 (USB_D+), U12.1 (I/O1), U12.6 (I/O1)
- net VBAT: now also U4.2 (CELL), U4.3 (VDD)
- net VSYS: now also C27.1, U2.10 (VDD), C19.2, C24.2, C25.2, C26.1, C28.2, R20.2, SW3.1, U11.7 (VDD), U11.8 (VDD), U3.10 (VIN_10)
- net at C11.2: now also U3.1 (VINA), U3.11 (VIN_11)
- net at M1.2 (-), U2.7 (OUT+): now also TP4.1
- net at M1.1 (+), U2.9 (OUT-): now also TP3.1
- net PGOOD: now reaches U10.7 (~{PGOOD})
- net PGOOD: now also U1.34 (IO41), R26.2
- net CHG_STAT: now reaches U10.9 (~{CHG})
- net CHG_STAT: now also U1.33 (IO40), R25.2
- net at R12.2, R13.1: now also U3.3 (FB)
- net I2S_LRCLK: now reaches U1.10 (IO17)
- net I2S_LRCLK: now also U11.14 (LRCLK)
- net FG_ALRT: now reaches U1.11 (IO18)
- net FG_ALRT: now also R29.1, U4.5 (~{ALERT})
- net BOOT: now reaches U1.27 (IO0)
- net BOOT: now also R24.2, SW2.1
- net at U1.3 (EN): now also C20.2, R23.2, SW1.1
- net SDCD: now reaches U1.35 (IO42)
- net SDCD: now also J1.4 (Pin_4)
- net RX: now reaches U1.36 (RXD0)
- net RX: now also TP2.1
- net TX: now reaches U1.37 (TXD0)
- net TX: now also TP1.1
- net PWR_SENSE: now reaches U1.38 (IO2)
- net PWR_SENSE: now also Q1.3 (D)
- net PWR_HOLD: now reaches U1.39 (IO1)
- net PWR_HOLD: now also D1.2
- net at U1.4 (IO4): now also R30.1
- net PDM_DATA: now reaches U1.5 (IO5)
- net PDM_DATA: now also J6.5 (Pin_5), J7.5 (Pin_5)
- net I2S_BCLK: now reaches U1.6 (IO6)
- net I2S_BCLK: now also U11.16 (BCLK)
- net I2S_DOUT: now reaches U1.8 (IO15)
- net I2S_DOUT: now also U11.1 (DIN)
- net AMP_SD: now reaches U1.9 (IO16)
- net AMP_SD: now also R22.1
- net at L2.1: now also U3.8 (L1_8), U3.9 (L1_9)
- net at L2.2: now also U3.6 (L2_6), U3.7 (L2_7)
- net at R14.2: now also U3.14 (PG)
- net +5V renamed VBUS
- net VBUS: now also U12.5 (VBUS)
- net CLK renamed SPI_CLK
- net SPI_CLK: now also J1.5 (Pin_5)
- net CS renamed OLED_CS
- net OLED_CS: now also J1.8 (Pin_8)
- net DC renamed OLED_DC
- net OLED_DC: now also J1.9 (Pin_9)
- net EN renamed HAPTICS_EN
- net MOSI renamed SPI_MOSI
- net SPI_MOSI: now also J1.6 (Pin_6)
- net RST renamed OLED_RST
- net OLED_RST: now also J1.10 (Pin_10)
- new net: R20.1, R21.1, U11.2 (GAIN_SLOT)
- new net: D1.1, Q1.1 (G), R28.2, SW3.2
- new net: D1.3, R27.2, U3.12 (EN)
- new net: LS1.2, U11.10 (OUTN)
- new net: R22.2, U11.4 (~{SD_MODE})
- new net: LS1.1, U11.9 (OUTP)
- new net PDM_CLK: J6.4 (Pin_4), J7.4 (Pin_4), R30.2
- no-connect marks 5 -> 14
Other:
- note added: "5v"
- note added: "Connector_JST:JST_PH_S2B-PH-K_1x02_P2.00mm_Horizontal"
- note added: "POWER"
- note added: "for 1200 mAH"
- note added: "make trach for Vbat thicker (0.5 mm)"
- note removed: "LRA actuator"
- note removed: "ROTARY AND FUEL GUADE HAVE THE SAME i2C address (0x36) so one needs to be on its own line"
- note removed: "add buttons for boot and reset"
- note removed: "decide gpio for ALRT"
- moved on the sheet: C10, C12, C13, C14, C15, C16, C17, J5, L2, R12, R13, R14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

Commit message: pcb changes
isolated certain parts for better layout configuration
Parts:
- R18: value 1.13k -> 1.78k
Changed lines of the file:
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@@
 			)
 		)
-		(property "Value" "1.13k"
+		(property "Value" "1.78k"
 			(at 479.806 223.52 0)
 			(show_name no)

Commit message: draft1pcb
draft 1 pcb schema
Parts:
- SW3: footprint Button_Switch_THT:SW_NKK_GW12LJP -> Button_Switch_SMD:SW_SPST_CK_KMS2xxGP
Connections:
- net MISO_SD: now also J1.5 (Pin_5); no longer J1.7 (Pin_7)
- net OLED_CS: now also J1.7 (Pin_7); no longer J1.8 (Pin_8)
- net OLED_RST: now also J1.8 (Pin_8); no longer J1.10 (Pin_10)
- net SDCS: now also J1.6 (Pin_6); no longer J1.11 (Pin_11)
- net SPI_CLK: now also J1.10 (Pin_10); no longer J1.5 (Pin_5)
- net SPI_MOSI: now also J1.11 (Pin_11); no longer J1.6 (Pin_6)
Changed lines of the file:
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@@
 	)
 	(label "OLED_CS"
-		(at 53.34 130.81 180)
+		(at 53.34 128.27 180)
 		(effects
 			(font
@@
 	)
 	(label "SDCS"
-		(at 53.34 138.43 180)
+		(at 53.34 125.73 180)
 		(effects
 			(font
@@
 	)
 	(label "OLED_RST"
-		(at 53.34 135.89 180)
+		(at 53.34 130.81 180)
 		(effects
 			(font
@@
 	)
 	(label "MISO_SD"
-		(at 53.34 128.27 180)
+		(at 53.34 123.19 180)
 		(effects
 			(font
@@
 	)
 	(label "SPI_CLK"
-		(at 53.34 123.19 180)
+		(at 53.34 135.89 180)
 		(effects
 			(font
@@
 	)
 	(label "SPI_MOSI"
-		(at 53.34 125.73 180)
+		(at 53.34 138.43 180)
 		(effects
 			(font
@@
 			)
 		)
-		(property "Footprint" "Button_Switch_THT:SW_NKK_GW12LJP"
+		(property "Footprint" "Button_Switch_SMD:SW_SPST_CK_KMS2xxGP"
 			(at 431.8 151.13 0)
 			(hide yes)

Commit message: changes
Parts:
- added D2, D3, D4, D5: LED, LED_SMD:LED_0805_2012Metric_Pad1.15x1.40mm_HandSolder, symbol Device:LED
- added H5: MountingHole, Connector_RJ:RJ45_Amphenol_RJMG1BD3B8K1ANR, symbol Mechanical:MountingHole
- added R4, R5, R6, R7: 1.5k, Resistor_SMD:R_0805_2012Metric_Pad1.20x1.40mm_HandSolder, symbol Device:R_US
- added TP6: SDA, TestPoint:TestPoint_THTPad_D1.5mm_Drill0.7mm, symbol Connector:TestPoint
- added TP7: SCL, TestPoint:TestPoint_THTPad_D1.5mm_Drill0.7mm, symbol Connector:TestPoint
- added TP8: FG_ALRT, TestPoint:TestPoint_THTPad_D1.5mm_Drill0.7mm, symbol Connector:TestPoint
Connections:
- net +3.3V: now also C27.1, C28.2, U2.10 (VDD), R6.1
- net CHG_STAT: now also D2.1 (K)
- net FG_ALRT: now also TP8.1
- net GND: now also D4.1 (K), D5.1 (K)
- net PGOOD: now also D3.1 (K)
- net SCL: now also TP7.1
- net SDA: now also TP6.1
- net VSYS: now also R4.2, R5.2; no longer C27.1, C28.2, U2.10 (VDD)
- net at U1.25 (IO48): now also R7.1
- new net: D2.2 (A), R4.1
- new net: D5.2 (A), R7.2
- new net: D4.2 (A), R6.2
- new net: D3.2 (A), R5.1
- no-connect marks 14 -> 13
Other:
- moved on the sheet: C26

Commit message: pre DRC final layout
Parts:
- removed H3, H4: MountingHole, MountingHole:MountingHole_2.2mm_M2, symbol Mechanical:MountingHole
- removed H5: MountingHole, Connector_RJ:RJ45_Amphenol_RJMG1BD3B8K1ANR, symbol Mechanical:MountingHole
- TP1, TP2, TP5, TP6, TP7, TP8: footprint TestPoint:TestPoint_THTPad_D1.5mm_Drill0.7mm -> TestPoint:TestPoint_Pad_D2.0mm
Changed lines of the file:
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@@
 			)
 		)
-		(property "Footprint" "TestPoint:TestPoint_THTPad_D1.5mm_Drill0.7mm"
+		(property "Footprint" "TestPoint:TestPoint_Pad_D2.0mm"
 			(at 38.1 234.95 0)
 			(hide yes)
@@
 	)
 	(symbol
-		(lib_id "Mechanical:MountingHole")
-		(at 22.86 281.94 0)
-		(unit 1)
-		(body_style 1)
-		(exclude_from_sim no)
-		(in_bom no)
-		(on_board yes)
-		(in_pos_files yes)
-		(dnp no)
-		(fields_autoplaced yes)
-		(property "Reference" "H5"
-			(at 25.4 280.6699 0)
-			(show_name no)
-			(do_not_autoplace no)
-			(effects
-				(font
-					(size 1.27 1.27)
-				)
-				(justify left)
-			)
-		)
-		(property "Value" "MountingHole"
-			(at 25.4 283.2099 0)
-			(show_name no)
-			(do_not_autoplace no)
-			(effects
-				(font
-					(size 1.27 1.27)
-				)
-				(justify left)
-			)
-		)
-		(property "Footprint" "Connector_RJ:RJ45_Amphenol_RJMG1BD3B8K1ANR"
-			(at 22.86 281.94 0)
-			(hide yes)
-			(show_name no)
-			(do_not_autoplace no)
-			(effects
-				(font
-					(size 1.27 1.27)
-				)
-			)
-		)
-		(property "Datasheet" ""
-			(at 22.86 281.94 0)
-			(hide yes)
-			(show_name no)
-			(do_not_autoplace no)
-			(effects
-				(font
-					(size 1.27 1.27)
-				)
-			)
-		)
-		(property "Description" "Mounting Hole without connection"
-			(at 22.86 281.94 0)
-			(hide yes)
-			(show_name no)
-			(do_not_autoplace no)
-			(effects
-				(font
-					(size 1.27 1.27)
-				)
-			)
-		)
-		(instances
-			(project "ESP32_PRELIM_DESIGN"
-				(path "/ad7b4e31-bbaa-4804-aa31-814eb5fa2fbb"
-					(reference "H5")
-					(unit 1)
-				)
-			)
-		)
-	)
-	(symbol
 		(lib_id "power:GND")
 		(at 501.65 242.57 0)
@@
 			)
 		)
-		(property "Footprint" "TestPoint:TestPoint_THTPad_D1.5mm_Drill0.7mm"
+		(property "Footprint" "TestPoint:TestPoint_Pad_D2.0mm"
 			(at 38.1 229.87 0)
 			(hide yes)
@@
 			)
 		)
-		(property "Footprint" "TestPoint:TestPoint_THTPad_D1.5mm_Drill0.7mm"
+		(property "Footprint" "TestPoint:TestPoint_Pad_D2.0mm"
 			(at 25.4 229.87 0)
 			(hide yes)
@@
 			)
 		)
-		(property "Footprint" "TestPoint:TestPoint_THTPad_D1.5mm_Drill0.7mm"
+		(property "Footprint" "TestPoint:TestPoint_Pad_D2.0mm"
 			(at 38.1 242.57 0)
 			(hide yes)
@@
 	)
 	(symbol
-		(lib_id "Mechanical:MountingHole")
-		(at 22.2134 271.0924 0)
-		(unit 1)
-		(body_style 1)
-		(exclude_from_sim no)
-		(in_bom no)
-		(on_board yes)
-		(in_pos_files yes)
-		(dnp no)
-		(fields_autoplaced yes)
-		(property "Reference" "H3"
-			(at 24.7534 269.8223 0)
-			(show_name no)
-			(do_not_autoplace no)
-			(effects
-				(font
-					(size 1.27 1.27)
-				)
-				(justify left)
-			)
-		)
-		(property "Value" "MountingHole"
-			(at 24.7534 272.3623 0)
-			(show_name no)
-			(do_not_autoplace no)
-			(effects
-				(font
-					(size 1.27 1.27)
-				)
-				(justify left)
-			)
-		)
-		(property "Footprint" "MountingHole:MountingHole_2.2mm_M2"
-			(at 22.2134 271.0924 0)
-			(hide yes)
-			(show_name no)
-			(do_not_autoplace no)
-			(effects
-				(font
-					(size 1.27 1.27)
-				)
-			)
-		)
-		(property "Datasheet" ""
-			(at 22.2134 271.0924 0)
-			(hide yes)
-			(show_name no)
-			(do_not_autoplace no)
-			(effects
-				(font
-					(size 1.27 1.27)
-				)
-			)
-		)
-		(property "Description" "Mounting Hole without connection"
-			(at 22.2134 271.0924 0)
-			(hide yes)
-			(show_name no)
-			(do_not_autoplace no)
-			(effects
-				(font
-					(size 1.27 1.27)
-				)
-			)
-		)
-		(instances
-			(project "ESP32_PRELIM_DESIGN"
-				(path "/ad7b4e31-bbaa-4804-aa31-814eb5fa2fbb"
-					(reference "H3")
-					(unit 1)
-				)
-			)
-		)
-	)
-	(symbol
 		(lib_id "Device:R_US")
 		(at 170.18 199.39 0)
@@
 			)
 		)
-		(property "Footprint" "TestPoint:TestPoint_THTPad_D1.5mm_Drill0.7mm"
+		(property "Footprint" "TestPoint:TestPoint_Pad_D2.0mm"
 			(at 25.4 240.03 0)
 			(hide yes)
@@
 			)
 		)
-		(property "Footprint" "TestPoint:TestPoint_THTPad_D1.5mm_Drill0.7mm"
+		(property "Footprint" "TestPoint:TestPoint_Pad_D2.0mm"
 			(at 25.4 234.95 0)
 			(hide yes)
@@
 					(unit 1)
 				)
-			)
-		)
-	)
-	(symbol
-		(lib_id "Mechanical:MountingHole")
-		(at 22.86 276.86 0)
-		(unit 1)
-		(body_style 1)
-		(exclude_from_sim no)
-		(in_bom no)
-		(on_board yes)
-		(in_pos_files yes)
-		(dnp no)
-		(fields_autoplaced yes)
-		(property "Reference" "H4"
-			(at 25.4 275.5899 0)
-			(show_name no)
-			(do_not_autoplace no)
-			(effects
-				(font
-					(size 1.27 1.27)
-				)
-				(justify left)
-			)
-		)
-		(property "Value" "MountingHole"
-			(at 25.4 278.1299 0)
-			(show_name no)
-			(do_not_autoplace no)
-			(effects
-				(font
-					(size 1.27 1.27)
-				)
-				(justify left)
-			)
-		)
-		(property "Footprint" "MountingHole:MountingHole_2.2mm_M2"
-			(at 22.86 276.86 0)
-			(hide yes)
-			(show_name no)
-			(do_not_autoplace no)
-			(effects
-				(font
-					(size 1.27 1.27)
-				)
-			)
-		)
-		(property "Datasheet" ""
-			(at 22.86 276.86 0)
-			(hide yes)
-			(show_name no)
-			(do_not_autoplace no)
-			(effects
-				(font
-					(size 1.27 1.27)
-				)
-			)
-		)
-		(property "Description" "Mounting Hole without connection"
-			(at 22.86 276.86 0)
-			(hide yes)
-			(show_name no)
-			(do_not_autoplace no)
-			(effects
-				(font
-					(size 1.27 1.27)
-				)
-			)
-		)
-		(instances
-			(project "ESP32_PRELIM_DESIGN"
-				(path "/ad7b4e31-bbaa-4804-aa31-814eb5fa2fbb"
-					(reference "H4")
-					(unit 1)
-				)

Commit message: final changes befpre pcb rev submission
Parts:
- R18: value 1.78k -> 2k
Changed lines of the file:
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@@
 		(dnp no)
 		(property "Reference" "R18"
-			(at 479.806 220.98 0)
+			(at 481.33 220.98 0)
 			(show_name no)
 			(do_not_autoplace no)
@@
 			)
 		)
-		(property "Value" "1.78k"
-			(at 479.806 223.52 0)
+		(property "Value" "2k"
+			(at 481.838 223.52 0)
 			(show_name no)
 			(do_not_autoplace no)

Commit message: final changes before CDR
Parts:
- renumbered C18 to C1, C13 to C10, C24 to C11, C10 to C12, C11 to C13, C22 to C16, C12 to C17, C16 to C18, C23 to C19, C27 to C2, C17 to C20, C28 to C3, C20 to C4, C1 to C5, C21 to C6, C26 to C7, C19 to C8, C25 to C9, D5 to D1, D4 to D2, D1 to D3, D2 to D4, D3 to D5, TP8 to FG_ALRT1, TP5 to GND1, J4 to J1, J1 to J2, J7 to J3, J6 to J4, L2 to L1, R2 to R1, R22 to R10, R6 to R11, R29 to R12, R28 to R13, R27 to R14, R12 to R19, R1 to R2, R19 to R20, R13 to R21, R25 to R22, R14 to R23, R4 to R24, R26 to R25, R5 to R26, R23 to R3, R30 to R4, R7 to R5, R24 to R6, R3 to R7, R20 to R8, R21 to R9, TP2 to RX1, TP7 to SCL1, TP6 to SDA1, TP3 to TP1, TP4 to TP2, TP1 to TX1, U2 to U1, U1 to U2, U11 to U3, U12 to U5, U3 to U6, U10 to U7

Commit message: final push (pk verified)
Parts:
- added H3: MountingHole, MountingHole:MountingHole_2.2mm_M2, symbol Mechanical:MountingHole
- R17: value 1.18k -> 3.3k
Connections:
- net +3.3V: now also R24.2, R26.2
- net VSYS: now also C13.2, U6.1 (VINA), U6.11 (VIN_11); no longer R24.2, R26.2
Changed lines of the file:
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@@
 	)
 	(junction
-		(at 529.59 198.12)
-		(diameter 0)
-		(color 0 0 0 0)
-	)
-	(junction
 		(at 515.62 110.49)
 		(diameter 0)
@@
 	(wire
 		(pts
-			(xy 523.24 198.12) (xy 529.59 198.12)
+			(xy 113.03 36.83) (xy 113.03 39.37)
 		)
 		(stroke
@@
 	(wire
 		(pts
-			(xy 113.03 36.83) (xy 113.03 39.37)
+			(xy 394.97 129.54) (xy 402.59 129.54)
 		)
 		(stroke
@@
 	(wire
 		(pts
-			(xy 394.97 129.54) (xy 402.59 129.54)
+			(xy 200.66 168.91) (xy 198.12 168.91)
 		)
 		(stroke
@@
 	(wire
 		(pts
-			(xy 200.66 168.91) (xy 198.12 168.91)
+			(xy 128.27 64.77) (xy 137.16 64.77)
 		)
 		(stroke
@@
 	(wire
 		(pts
-			(xy 128.27 64.77) (xy 137.16 64.77)
+			(xy 467.36 113.03) (xy 467.36 116.84)
 		)
 		(stroke
@@
 	(wire
 		(pts
-			(xy 467.36 113.03) (xy 467.36 116.84)
+			(xy 467.36 110.49) (xy 467.36 113.03)
 		)
 		(stroke
@@
 		)
 	)
+	(junction
+		(at 467.36 113.03)
+		(diameter 0)
+		(color 0 0 0 0)
+	)
 	(wire
 		(pts
@@
 	)
 	(label "VSYS"
-		(at 541.02 198.12 0)
+		(at 523.24 198.12 0)
 		(effects
 			(font
@@
 	)
 	(symbol
+		(lib_id "power:+3.3V")
+		(at 541.02 198.12 0)
+		(unit 1)
+		(body_style 1)
+		(exclude_from_sim no)
+		(in_bom yes)
+		(on_board yes)
+		(in_pos_files yes)
+		(dnp no)
+		(fields_autoplaced yes)
+		(property "Reference" "#PWR069"
+			(at 541.02 201.93 0)
+			(hide yes)
+			(show_name no)
+			(do_not_autoplace no)
+			(effects
+				(font
+					(size 1.27 1.27)
+				)
+			)
+		)
+		(property "Value" "+3.3V"
+			(at 541.02 194.31 0)
+			(show_name no)
+			(do_not_autoplace no)
+			(effects
+				(font
+					(size 1.27 1.27)
+				)
+			)
+		)
+		(property "Footprint" ""
+			(at 541.02 198.12 0)
+			(hide yes)
+			(show_name no)
+			(do_not_autoplace no)
+			(effects
+				(font
+					(size 1.27 1.27)
+				)
+			)
+		)
+		(property "Datasheet" ""
+			(at 541.02 198.12 0)
+			(hide yes)
+			(show_name no)
+			(do_not_autoplace no)
+			(effects
+				(font
+					(size 1.27 1.27)
+				)
+			)
+		)
+		(property "Description" "Power symbol creates a global label with name \"+3.3V\""
+			(at 541.02 198.12 0)
+			(hide yes)
+			(show_name no)
+			(do_not_autoplace no)
+			(effects
+				(font
+					(size 1.27 1.27)
+				)
+			)
+		)
+		(pin "1"
+		)
+		(instances
+			(project "ESP32_PRELIM_DESIGN"
+				(path "/ad7b4e31-bbaa-4804-aa31-814eb5fa2fbb"
+					(reference "#PWR069")
+					(unit 1)
+				)
+			)
+		)
+	)
+	(symbol
 		(lib_id "Device:LED")
 		(at 529.59 185.42 270)
@@
 			)
 		)
-		(property "Value" "1.18k"
+		(property "Value" "3.3k"
 			(at 472.186 223.52 0)
 			(show_name no)
@@
 					(unit 1)
 				)
+			)
+		)
+	)
+	(symbol
+		(lib_id "Mechanical:MountingHole")
+		(at 21.59 271.78 0)
+		(unit 1)
+		(body_style 1)
+		(exclude_from_sim no)
+		(in_bom no)
+		(on_board yes)
+		(in_pos_files yes)
+		(dnp no)
+		(fields_autoplaced yes)
+		(property "Reference" "H3"
+			(at 24.13 270.5099 0)
+			(show_name no)
+			(do_not_autoplace no)
+			(effects
+				(font
+					(size 1.27 1.27)
+				)
+				(justify left)
+			)
+		)
+		(property "Value" "MountingHole"
+			(at 24.13 273.0499 0)
+			(show_name no)
+			(do_not_autoplace no)
+			(effects
+				(font
+					(size 1.27 1.27)
+				)
+				(justify left)
+			)
+		)
+		(property "Footprint" "MountingHole:MountingHole_2.2mm_M2"
+			(at 21.59 271.78 0)
+			(hide yes)
+			(show_name no)
+			(do_not_autoplace no)
+			(effects
+				(font
+					(size 1.27 1.27)
+				)
+			)
+		)
+		(property "Datasheet" ""
+			(at 21.59 271.78 0)
+			(hide yes)
+			(show_name no)
+			(do_not_autoplace no)
+			(effects
+				(font
+					(size 1.27 1.27)
+				)
+			)
+		)
+		(property "Description" "Mounting Hole without connection"
+			(at 21.59 271.78 0)
+			(hide yes)
+			(show_name no)
+			(do_not_autoplace no)
+			(effects
+				(font
+					(size 1.27 1.27)
+				)
+			)
+		)
+		(instances
+			(project "ESP32_PRELIM_DESIGN"
+				(path "/ad7b4e31-bbaa-4804-aa31-814eb5fa2fbb"
+					(reference "H3")
+					(unit 1)
+				)
